File: K9HZ_LPF_Module/K9HZ_LPF_V1.00_Schematics/K9HZ_100W_11band_LPF-Filter/K9HZ_100W_11band_LPF-Filter.kicad_sch (KiCad schematic)
At the start: 169 parts, among them J17 RF interconnect, J22 RF interconnect, J26 LPF CTRL LOW, J27 LPF CTRL HI, K10 HF41F/12-ZS, K11 HF41F/12-ZS, K12 HF41F/12-ZS, K13 HF41F/12-ZS, K14 HF41F/12-ZS, K15 HF41F/12-ZS, K16 HF41F/12-ZS, K17 HF41F/12-ZS, K18 HF41F/12-ZS, K19 HF41F/12-ZS, K20 HF41F/12-ZS, K21 HF41F/12-ZS, K22 HF41F/12-ZS, K23 HF41F/12-ZS, K24 HF41F/12-ZS, K25 HF41F/12-ZS, K26 HF41F/12-ZS, K27 HF41F/12-ZS, K28 HF41F/12-ZS, K29 HF41F/12-ZS, K32 HF41F/12-ZS, K33 HF41F/12-ZS, K8 HF41F/12-ZS, K9 HF41F/12-ZS

Commit message: Changed LPF to use 1206 and 0805
LPF has multiple changes but all to support use of either 1206 or 0805 caps
Parts:
- added H3, H4: ~, MountingHole:MountingHole_3.2mm_M3_DIN965_Pad, symbol Mechanical:MountingHole_Pad
- C1: renamed from C107; footprint Capacitor_SMD:C_1206_3216Metric -> T41_Library:C_1206_0805_Dual
- C10: renamed from C102; footprint Capacitor_SMD:C_1206_3216Metric -> T41_Library:C_1206_0805_Dual
- C100: renamed from C39; footprint Capacitor_SMD:C_1206_3216Metric -> T41_Library:C_1206_0805_Dual
- C101: renamed from C51; footprint Capacitor_SMD:C_1206_3216Metric -> T41_Library:C_1206_0805_Dual
- C102: renamed from C82; footprint Capacitor_SMD:C_1206_3216Metric -> T41_Library:C_1206_0805_Dual
- C103: renamed from C100; footprint Capacitor_SMD:C_1206_3216Metric -> T41_Library:C_1206_0805_Dual
- C104: renamed from C70; footprint Capacitor_SMD:C_1206_3216Metric -> T41_Library:C_1206_0805_Dual
- C105: renamed from C157; footprint Capacitor_SMD:C_1206_3216Metric -> T41_Library:C_1206_0805_Dual
- C106: renamed from C158; footprint Capacitor_SMD:C_1206_3216Metric -> T41_Library:C_1206_0805_Dual
- C11: renamed from C59; footprint Capacitor_SMD:C_1206_3216Metric -> T41_Library:C_1206_0805_Dual
- C12: renamed from C60; footprint Capacitor_SMD:C_1206_3216Metric -> T41_Library:C_1206_0805_Dual
- C13: renamed from C108; footprint Capacitor_SMD:C_1206_3216Metric -> T41_Library:C_1206_0805_Dual
- C14: renamed from C109; footprint Capacitor_SMD:C_1206_3216Metric -> T41_Library:C_1206_0805_Dual
- C15: renamed from C26; footprint Capacitor_SMD:C_1206_3216Metric -> T41_Library:C_1206_0805_Dual
- C16: renamed from C30; footprint Capacitor_SMD:C_1206_3216Metric -> T41_Library:C_1206_0805_Dual
- C17: renamed from C46; footprint Capacitor_SMD:C_1206_3216Metric -> T41_Library:C_1206_0805_Dual
- C18: renamed from C56; footprint Capacitor_SMD:C_1206_3216Metric -> T41_Library:C_1206_0805_Dual
- C19: renamed from C76; footprint Capacitor_SMD:C_1206_3216Metric -> T41_Library:C_1206_0805_Dual
- C2: renamed from C106; footprint Capacitor_SMD:C_1206_3216Metric -> T41_Library:C_1206_0805_Dual
- C20: renamed from C86; footprint Capacitor_SMD:C_1206_3216Metric -> T41_Library:C_1206_0805_Dual
- C21: renamed from C92; footprint Capacitor_SMD:C_1206_3216Metric -> T41_Library:C_1206_0805_Dual
- C22: renamed from C101; footprint Capacitor_SMD:C_1206_3216Metric -> T41_Library:C_1206_0805_Dual
- C23: renamed from C61; footprint Capacitor_SMD:C_1206_3216Metric -> T41_Library:C_1206_0805_Dual
- C24: renamed from C62; footprint Capacitor_SMD:C_1206_3216Metric -> T41_Library:C_1206_0805_Dual
- C25: renamed from C110; footprint Capacitor_SMD:C_1206_3216Metric -> T41_Library:C_1206_0805_Dual
- C26: renamed from C111; footprint Capacitor_SMD:C_1206_3216Metric -> T41_Library:C_1206_0805_Dual
- C27: renamed from C31; footprint Capacitor_SMD:C_1206_3216Metric -> T41_Library:C_1206_0805_Dual
- C28: renamed from C40; footprint Capacitor_SMD:C_1206_3216Metric -> T41_Library:C_1206_0805_Dual
- C29: renamed from C44; footprint Capacitor_SMD:C_1206_3216Metric -> T41_Library:C_1206_0805_Dual
- C3: renamed from C28; footprint Capacitor_SMD:C_1206_3216Metric -> T41_Library:C_1206_0805_Dual
- C30: renamed from C57; footprint Capacitor_SMD:C_1206_3216Metric -> T41_Library:C_1206_0805_Dual
- C31: renamed from C75; footprint Capacitor_SMD:C_1206_3216Metric -> T41_Library:C_1206_0805_Dual
- C32: renamed from C87; footprint Capacitor_SMD:C_1206_3216Metric -> T41_Library:C_1206_0805_Dual
- C33: renamed from C89; footprint Capacitor_SMD:C_1206_3216Metric -> T41_Library:C_1206_0805_Dual
- C34: renamed from C93; footprint Capacitor_SMD:C_1206_3216Metric -> T41_Library:C_1206_0805_Dual
- C35: renamed from C66; footprint Capacitor_SMD:C_1206_3216Metric -> T41_Library:C_1206_0805_Dual
- C36: renamed from C67; footprint Capacitor_SMD:C_1206_3216Metric -> T41_Library:C_1206_0805_Dual
- C37: renamed from C112; footprint Capacitor_SMD:C_1206_3216Metric -> T41_Library:C_1206_0805_Dual
- C38: renamed from C113; footprint Capacitor_SMD:C_1206_3216Metric -> T41_Library:C_1206_0805_Dual
- C39: renamed from C25; footprint Capacitor_SMD:C_1206_3216Metric -> T41_Library:C_1206_0805_Dual
- C4: renamed from C29; footprint Capacitor_SMD:C_1206_3216Metric -> T41_Library:C_1206_0805_Dual
- C40: renamed from C32; footprint Capacitor_SMD:C_1206_3216Metric -> T41_Library:C_1206_0805_Dual
- C41: renamed from C43; footprint Capacitor_SMD:C_1206_3216Metric -> T41_Library:C_1206_0805_Dual
- C42: renamed from C54; footprint Capacitor_SMD:C_1206_3216Metric -> T41_Library:C_1206_0805_Dual
- C43: renamed from C73; footprint Capacitor_SMD:C_1206_3216Metric -> T41_Library:C_1206_0805_Dual
- C44: renamed from C88; footprint Capacitor_SMD:C_1206_3216Metric -> T41_Library:C_1206_0805_Dual
- C45: renamed from C94; footprint Capacitor_SMD:C_1206_3216Metric -> T41_Library:C_1206_0805_Dual
- C46: renamed from C103; footprint Capacitor_SMD:C_1206_3216Metric -> T41_Library:C_1206_0805_Dual
- C47: renamed from C58; footprint Capacitor_SMD:C_1206_3216Metric -> T41_Library:C_1206_0805_Dual
- C48: renamed from C114; footprint Capacitor_SMD:C_1206_3216Metric -> T41_Library:C_1206_0805_Dual
- C49: renamed from C115; footprint Capacitor_SMD:C_1206_3216Metric -> T41_Library:C_1206_0805_Dual
- C5: renamed from C45; footprint Capacitor_SMD:C_1206_3216Metric -> T41_Library:C_1206_0805_Dual
- C50: renamed from C27; footprint Capacitor_SMD:C_1206_3216Metric -> T41_Library:C_1206_0805_Dual
- C51: renamed from C33; footprint Capacitor_SMD:C_1206_3216Metric -> T41_Library:C_1206_0805_Dual
- C52: renamed from C47; footprint Capacitor_SMD:C_1206_3216Metric -> T41_Library:C_1206_0805_Dual
- C53: renamed from C78; footprint Capacitor_SMD:C_1206_3216Metric -> T41_Library:C_1206_0805_Dual
- C54: renamed from C95; footprint Capacitor_SMD:C_1206_3216Metric -> T41_Library:C_1206_0805_Dual
- C55: renamed from C104; footprint Capacitor_SMD:C_1206_3216Metric -> T41_Library:C_1206_0805_Dual
- C56: renamed from C68; footprint Capacitor_SMD:C_1206_3216Metric -> T41_Library:C_1206_0805_Dual
- C57: renamed from C116; footprint Capacitor_SMD:C_1206_3216Metric -> T41_Library:C_1206_0805_Dual
- C58: renamed from C117; footprint Capacitor_SMD:C_1206_3216Metric -> T41_Library:C_1206_0805_Dual
- C59: renamed from C34; footprint Capacitor_SMD:C_1206_3216Metric -> T41_Library:C_1206_0805_Dual
- C6: renamed from C55; footprint Capacitor_SMD:C_1206_3216Metric -> T41_Library:C_1206_0805_Dual
- C60: renamed from C48; footprint Capacitor_SMD:C_1206_3216Metric -> T41_Library:C_1206_0805_Dual
- C61: renamed from C79; footprint Capacitor_SMD:C_1206_3216Metric -> T41_Library:C_1206_0805_Dual
- C62: renamed from C96; footprint Capacitor_SMD:C_1206_3216Metric -> T41_Library:C_1206_0805_Dual
- C63: renamed from C64; footprint Capacitor_SMD:C_1206_3216Metric -> T41_Library:C_1206_0805_Dual
- C64: renamed from C118; footprint Capacitor_SMD:C_1206_3216Metric -> T41_Library:C_1206_0805_Dual
- C65: renamed from C119; footprint Capacitor_SMD:C_1206_3216Metric -> T41_Library:C_1206_0805_Dual
- C66: renamed from C24; footprint Capacitor_SMD:C_1206_3216Metric -> T41_Library:C_1206_0805_Dual
- C67: renamed from C35; footprint Capacitor_SMD:C_1206_3216Metric -> T41_Library:C_1206_0805_Dual
- C68: renamed from C42; footprint Capacitor_SMD:C_1206_3216Metric -> T41_Library:C_1206_0805_Dual
- C69: renamed from C52; footprint Capacitor_SMD:C_1206_3216Metric -> T41_Library:C_1206_0805_Dual
- C7: renamed from C77; footprint Capacitor_SMD:C_1206_3216Metric -> T41_Library:C_1206_0805_Dual
- C70: renamed from C74; footprint Capacitor_SMD:C_1206_3216Metric -> T41_Library:C_1206_0805_Dual
- C71: renamed from C83; footprint Capacitor_SMD:C_1206_3216Metric -> T41_Library:C_1206_0805_Dual
- C72: renamed from C90; footprint Capacitor_SMD:C_1206_3216Metric -> T41_Library:C_1206_0805_Dual
- C73: renamed from C105; footprint Capacitor_SMD:C_1206_3216Metric -> T41_Library:C_1206_0805_Dual
- C74: renamed from C71; footprint Capacitor_SMD:C_1206_3216Metric -> T41_Library:C_1206_0805_Dual
- C75: renamed from C120; footprint Capacitor_SMD:C_1206_3216Metric -> T41_Library:C_1206_0805_Dual
- C76: renamed from C121; footprint Capacitor_SMD:C_1206_3216Metric -> T41_Library:C_1206_0805_Dual
- C77: renamed from C36; footprint Capacitor_SMD:C_1206_3216Metric -> T41_Library:C_1206_0805_Dual
- C78: renamed from C49; footprint Capacitor_SMD:C_1206_3216Metric -> T41_Library:C_1206_0805_Dual
- C79: renamed from C80; footprint Capacitor_SMD:C_1206_3216Metric -> T41_Library:C_1206_0805_Dual
- C8: renamed from C84; footprint Capacitor_SMD:C_1206_3216Metric -> T41_Library:C_1206_0805_Dual
- C80: renamed from C97; footprint Capacitor_SMD:C_1206_3216Metric -> T41_Library:C_1206_0805_Dual
- C81: renamed from C65; footprint Capacitor_SMD:C_1206_3216Metric -> T41_Library:C_1206_0805_Dual
- C82: renamed from C122; footprint Capacitor_SMD:C_1206_3216Metric -> T41_Library:C_1206_0805_Dual
- C83: renamed from C123; footprint Capacitor_SMD:C_1206_3216Metric -> T41_Library:C_1206_0805_Dual
- C84: renamed from C37; footprint Capacitor_SMD:C_1206_3216Metric -> T41_Library:C_1206_0805_Dual
- C85: renamed from C50; footprint Capacitor_SMD:C_1206_3216Metric -> T41_Library:C_1206_0805_Dual
- C86: renamed from C81; footprint Capacitor_SMD:C_1206_3216Metric -> T41_Library:C_1206_0805_Dual
- C87: renamed from C98; footprint Capacitor_SMD:C_1206_3216Metric -> T41_Library:C_1206_0805_Dual
- C88: renamed from C63; footprint Capacitor_SMD:C_1206_3216Metric -> T41_Library:C_1206_0805_Dual
- C89: renamed from C124; footprint Capacitor_SMD:C_1206_3216Metric -> T41_Library:C_1206_0805_Dual
- C9: renamed from C91; footprint Capacitor_SMD:C_1206_3216Metric -> T41_Library:C_1206_0805_Dual
- C90: renamed from C125; footprint Capacitor_SMD:C_1206_3216Metric -> T41_Library:C_1206_0805_Dual
- C91: renamed from C38; footprint Capacitor_SMD:C_1206_3216Metric -> T41_Library:C_1206_0805_Dual
- C92: renamed from C41; footprint Capacitor_SMD:C_1206_3216Metric -> T41_Library:C_1206_0805_Dual
- C93: renamed from C53; footprint Capacitor_SMD:C_1206_3216Metric -> T41_Library:C_1206_0805_Dual
- C94: renamed from C72; footprint Capacitor_SMD:C_1206_3216Metric -> T41_Library:C_1206_0805_Dual
- C95: renamed from C85; footprint Capacitor_SMD:C_1206_3216Metric -> T41_Library:C_1206_0805_Dual
- C96: renamed from C99; footprint Capacitor_SMD:C_1206_3216Metric -> T41_Library:C_1206_0805_Dual
- C97: renamed from C69; footprint Capacitor_SMD:C_1206_3216Metric -> T41_Library:C_1206_0805_Dual
- C98: renamed from C126; footprint Capacitor_SMD:C_1206_3216Metric -> T41_Library:C_1206_0805_Dual
- C99: renamed from C127; footprint Capacitor_SMD:C_1206_3216Metric -> T41_Library:C_1206_0805_Dual
- H1: renamed from H5; footprint MountingHole:MountingHole_4.3mm_M4_DIN965_Pad -> MountingHole:MountingHole_3.2mm_M3_DIN965_Pad
- H2: renamed from H6; footprint MountingHole:MountingHole_4.3mm_M4_DIN965_Pad -> MountingHole:MountingHole_3.2mm_M3_DIN965_Pad
- renumbered J22 to J1, J17 to J2, J26 to J3, J27 to J4, K16 to K1, K23 to K10, K15 to K11, K24 to K12, K9 to K13, K25 to K14, K8 to K15, K26 to K16, K10 to K17, K27 to K18, K11 to K19, K21 to K2, K28 to K20, K18 to K21, K29 to K22, K33 to K23, K32 to K24, K14 to K3, K19 to K4, K13 to K5, K20 to K6, K12 to K7, K22 to K8, K17 to K9, L3 to L1, L6 to L10, L17 to L11, L28 to L12, L7 to L13, L18 to L14, L29 to L15, L8 to L16, L19 to L17, L30 to L18, L9 to L19, L14 to L2, L31 to L21, L10 to L22, L21 to L23, L32 to L24, L11 to L25, L22 to L26, L33 to L27, L12 to L28, L23 to L29, L25 to L3, L34 to L30, L13 to L31, L24 to L32, L35 to L33, L15 to L5, L26 to L6, L5 to L7, L16 to L8, L27 to L9
Connections:
- net GND: now also H3.1, H4.1
Other:
- moved on the sheet: H1, H2
